File: templates/schematic-template.kicad_sch (KiCad schematic)
At the start: 0 parts

Commit message: chore(library): add KiCad project template files so init-feature.sh scaffolds correctly
Agent-Logs-Url: https://github.com/rockett90/hardware-features/sessions/12fcd6ee-ba3a-4fda-bdc8-88da143073d0

Co-authored-by: rockett90 <149118299+rockett90@users.noreply.github.com>
Other:
- title: FEATURE_NAME -> (none)
Changed lines of the file:
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@@
 (kicad_sch
-	(version 20260306)
-	(generator "eeschema")
-	(generator_version "10.0")
-	(paper "A3")
-	(title_block
-		(title "FEATURE_NAME")
-		(date "YYYY-MM-DD")
-		(rev "0.1")
-		(company "")
-		(comment 1 "Replace FEATURE_NAME with the actual feature name")
-	)
-	(sheet_instances
-		(path "/"
-			(page "1")
-		)
-	)
+  (version 20231120)
+  (generator eeschema)
+  (generator_version 8.0)
+  (paper "A3")
+  (title_block
+    (title "")
+    (date "")
+    (rev "A")
+    (company "")
+    (comment 1 "")
+    (comment 2 "")
+    (comment 3 "")
+    (comment 4 "")
+  )
+  (sheet_instances
+    (path "/" (page "1"))
+  )
 )
