File: features/simple-amplifier/simple-amplifier.kicad_sch (KiCad schematic)
At the start: 0 parts

Commit message: chore(simple-amplifier): add first schematic
Other:
- added sheet amplifier (amplifier.kicad_sch)
- added sheet buffer (buffer.kicad_sch)
